Commit message: Add rgbd camera to my robot

File: my_robot/urdf/my_robot.xacro (robot description, xacro)
@@ -197,3 +197,12 @@
     <material>Gazebo/Black</material>
   </gazebo>
+  <!--RGBD Camera joint-->
+  <joint name="camera_optical_joint" type="fixed">
+    <origin xyz="0 0 0" rpy="-1.5707 0 -1.5707"/>
+    <parent link="camera"/>
+    <child link="camera_link_optical"/>
+  </joint>
+  <!--RGBD Camera-->
+  <link name="camera_link_optical">
+  </link>
 </robot>
